File: debouncer.kicad_pcb (KiCad board)
At the start: 2 copper layers, 15 parts, among them J1 Conn_01x14_Male, J2 Conn_01x06_Male, U1 74HC14

Commit message: 05-10
Parts:
- C1, C2, C3, C4, C5, C6: footprint Capacitors_SMD:C_1206_HandSoldering -> Capacitor_SMD:C_1206_3216Metric_Pad1.42x1.75mm_HandSolder
- J1: value Conn_01x14_Male -> Conn_02x07_Row_Letter_Last; footprint Pin_Headers:Pin_Header_Straight_1x14_Pitch2.54mm -> Connector_PinHeader_2.54mm:PinHeader_2x07_P2.54mm_Vertical
- J2: footprint Pin_Headers:Pin_Header_Straight_1x06_Pitch2.54mm -> Connector_PinHeader_2.54mm:PinHeader_1x06_P2.54mm_Vertical
- R1, R2, R3, R4, R5, R6: footprint Resistors_SMD:R_1206_HandSoldering -> Resistor_SMD:R_1206_3216Metric_Pad1.42x1.75mm_HandSolder
- U1: footprint SMD_Packages:SOIC-14_N -> Package_SO:SOIC-14_3.9x8.7mm_P1.27mm
- moved J1 130.1 mm to (109.2, 129.5), turned to 90 degrees
- moved C4 128.5 mm to (90.2, 121.9)
- moved C2 113.8 mm to (87.6, 110.5), turned to 0 degrees
- moved R6 110.7 mm to (115.6, 137.2), turned to 180 degrees
- moved C5 104.9 mm to (89.1, 128.3), turned to 0 degrees
- moved C6 104.5 mm to (86.6, 104.1)
- moved U1 97.3 mm to (111.8, 113.0), turned to 0 degrees
- moved J2 96.6 mm to (106.7, 88.9)
- moved C3 90.9 mm to (90.4, 116.8), turned to 0 degrees
- moved R1 86.1 mm to (122.8, 90.3), turned to 0 degrees
- moved R4 76.4 mm to (130.3, 83.2)
- moved C1 76.4 mm to (98.0, 109.2), turned to 0 degrees
- moved R5 46.4 mm to (156.2, 102.9)
- moved R2 45.4 mm to (157.3, 76.2)
- moved R3 35.9 mm to (154.7, 88.9), turned to 0 degrees
Connections:
- C1 pad 1: +5V -> Net-(C1-Pad1)
- C2 pad 1: +5V -> Net-(C2-Pad1)
- C3 pad 1: +5V -> Net-(C3-Pad1)
- C4 pad 1: +5V -> Net-(C4-Pad1)
- C5 pad 1: +5V -> Net-(C5-Pad1)
- C6 pad 1: +5V -> Net-(C6-Pad1)
- J1 pad 1: Net-(C1-Pad2) -> Net-(C1-Pad1)
- J1 pad 10: +5V -> Net-(C5-Pad2)
- J1 pad 11: Net-(C6-Pad2) -> Net-(C6-Pad1)
- J1 pad 12: +5V -> Net-(C6-Pad2)
- J1 pad 13: +5V -> VDC
- J1 pad 2: +5V -> Net-(C1-Pad2)
- J1 pad 3: Net-(C2-Pad2) -> Net-(C2-Pad1)
- J1 pad 4: +5V -> Net-(C2-Pad2)
- J1 pad 5: Net-(C3-Pad2) -> Net-(C3-Pad1)
- J1 pad 6: +5V -> Net-(C3-Pad2)
- J1 pad 7: Net-(C4-Pad2) -> Net-(C4-Pad1)
- J1 pad 8: +5V -> Net-(C4-Pad2)
- J1 pad 9: Net-(C5-Pad2) -> Net-(C5-Pad1)
- U1 pad 14: GND -> VDC
- U1 pad 7: +5V -> GND
Routing:
- net Net-(C1-Pad2): track 0.00 -> 29.4 mm
- net Net-(C1-Pad1): track 0.00 -> 26.4 mm
Other:
- net class My added: clearance 0.5, trace_width 0.5, via_dia 0.8, via_drill 0.4
