File: debouncer.sch (KiCad schematic (older format))
At the start: 15 parts, among them J2 Conn_01x06_Male, U1 74HC14

Commit message: 05-10
Parts:
- C1, C2, C3, C4, C5, C6: footprint Capacitors_SMD:C_1206_HandSoldering -> Capacitor_SMD:C_1206_3216Metric_Pad1.42x1.75mm_HandSolder
- J1: renamed from J?; footprint (none) -> Connector_PinHeader_2.54mm:PinHeader_2x07_P2.54mm_Vertical; symbol Connector_Generic:Conn_02x07_Row_Letter_Last -> Connector_Generic:Conn_02x07_Odd_Even
- J2: footprint Pin_Headers:Pin_Header_Straight_1x06_Pitch2.54mm -> Connector_PinHeader_2.54mm:PinHeader_1x06_P2.54mm_Vertical
- R1, R2, R3, R4, R5, R6: footprint Resistors_SMD:R_1206_HandSoldering -> Resistor_SMD:R_1206_3216Metric_Pad1.42x1.75mm_HandSolder
- U1: footprint (none) -> Package_SO:SOIC-14_3.9x8.7mm_P1.27mm
- U1: footprint SMD_Packages:SOIC-14_N -> Package_SO:SOIC-14_3.9x8.7mm_P1.27mm
Connections:
- wire segments 74 -> 100
